File: kicad/tester.kicad_pcb (KiCad board)
At the start: 2 copper layers, 67 x 21 mm, 71 parts, among them J3 CONN_01X06, Q1 IRLML2402, Q2 IRLML6402, Q3 BC847, Q4 BC847, Q5 BC847, U1 OLED_128x64, U2 NCP1450A, U3 ATMEGA328-AU, U4 LTC4054, U5 74LVC1G17, U6 SRV05, U7 XC6206P332, U8 MICRO-B_USB, Y1 16MHz

Commit message: Continue work with pcb
Parts:
- D2: footprint TO_SOT_Packages_SMD:SOT-23 -> LEDs:LED_D3.0mm; moved to B.Cu
- moved R8 42.3 mm to (252.0, 76.0), turned to 270 degrees
- moved C10 40.4 mm to (254.5, 75.2), turned to 0 degrees
- moved Q3 38.6 mm to (249.0, 73.2), turned to 180 degrees
- moved L1 36.9 mm to (266.5, 63.5), turned to 180 degrees
- moved R9 36.7 mm to (252.0, 73.0), turned to 270 degrees
- moved D1 32.2 mm to (265.5, 73.8), turned to 0 degrees
- moved U2 28.1 mm to (256.2, 64.8)
- moved Q1 28.0 mm to (260.8, 64.8)
- moved C1 27.6 mm to (255.0, 68.5), turned to 270 degrees
- moved C2 21.8 mm to (252.0, 67.2), turned to 90 degrees
- moved D2 16.7 mm to (248.0, 69.8), turned to 90 degrees
- moved R16 14.9 mm to (209.5, 63.0), turned to 270 degrees
- moved R14 14.5 mm to (215.0, 63.0), turned to 270 degrees
- moved R15 13.8 mm to (212.2, 63.0), turned to 270 degrees
- moved R19 12.6 mm to (210.8, 73.0), turned to 0 degrees
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Routing:
- net Net-(D2-Pad2): track 0.00 -> 14.2 mm
- net Net-(D1-Pad2): track 0.00 -> 14.1 mm
- net Net-(J1-Pad2): track 0.00 -> 12.6 mm
- net VCC: track 2.15 -> 14.4 mm
- net GND: track 73.6 -> 85.5 mm
- net Net-(J1-Pad1): track 0.00 -> 10.8 mm
- net Net-(J1-Pad3): track 0.00 -> 9.12 mm
- net Net-(R16-Pad2): track 0.00 -> 8.77 mm
- net /BATT_TEST: track 4.01 -> 10.7 mm, vias 0 -> 1
- net Net-(R15-Pad2): track 0.00 -> 5.94 mm
- net Net-(C10-Pad1): track 0.00 -> 5.39 mm
- net Net-(C15-Pad2): track 13.7 -> 19.0 mm
- net /MOSI: track 0.00 -> 4.27 mm
- net Net-(R14-Pad2): track 0.00 -> 3.96 mm
- net Net-(D2-Pad1): track 0.00 -> 3.45 mm
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