File: kicad/tester.kicad_pcb (KiCad board)
At the start: 2 copper layers, 67 x 21 mm, 71 parts, among them J3 CONN_01X06, Q1 IRLML2402, Q2 IRLML6402, Q3 BC847, Q4 BC847, Q5 BC847, U1 OLED_128x64, U2 NCP1450A, U3 ATMEGA328-AU, U4 LTC4054, U5 74LVC1G17, U6 SRV05, U7 XC6206P332, U8 MICRO-B_USB, Y1 16MHz

Commit message: update pcb
Parts:
- Y1: moved to B.Cu
- moved Y1 102.8 mm to (232.2, 66.2), turned to 90 degrees
- moved D5 72.1 mm to (244.8, 77.8), turned to 270 degrees
- moved J3 57.9 mm to (211.9, 76.5), turned to 180 degrees
- moved D7 48.1 mm to (220.8, 78.8)
- moved R11 37.6 mm to (221.6, 61.8), turned to 90 degrees
- moved R13 34.0 mm to (220.4, 57.2), turned to 90 degrees
- moved Q4 31.3 mm to (218.2, 62.2), turned to 270 degrees
Connections:
- J3 pad 2: VCC -> Net-(C7-Pad1)
Routing:
- net /RES: track 0.00 -> 23.4 mm
- net Net-(C7-Pad1): track 0.00 -> 18.8 mm
- net Net-(C12-Pad2): track 0.00 -> 16.6 mm
- net Net-(C11-Pad2): track 0.00 -> 13.8 mm
- net GND: track 85.5 -> 99.1 mm
- net /MOSI: track 4.27 -> 15.5 mm
- net /HV: track 1.75 -> 9.72 mm
- net /SCK: track 3.32 -> 6.95 mm

Commit message: Working with pcb
Parts:
- C16, C3, C4, C5, C6, R1, R2, R3, R4, R5, U1, U7: moved to B.Cu
- moved C13 102.5 mm to (179.7, 66.0)
- moved D3 102.5 mm to (175.9, 66.0)
- moved R12 102.5 mm to (175.9, 69.8)
- moved R21 64.3 mm to (178.4, 86.3)
- moved R22 64.3 mm to (191.7, 82.3)
- moved C11 57.7 mm to (217.8, 102.1)
- moved C12 57.7 mm to (224.5, 107.2)
- moved R10 57.7 mm to (189.2, 106.3)
- moved C7 57.7 mm to (231.6, 97.1)
- moved L2 57.7 mm to (212.8, 100.1)
- moved C8 57.7 mm to (224.8, 102.1)
- moved C14 57.7 mm to (224.5, 97.1)
- moved C3 47.5 mm to (223.5, 70.0), turned to 90 degrees
- moved C4 44.8 mm to (225.5, 70.0), turned to 90 degrees
- moved C16 42.3 mm to (227.5, 70.0), turned to 90 degrees
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Routing:
- net GND: track 99.1 -> 153.0 mm
- net /RES: track 23.4 -> 0.00 mm
- net Net-(C7-Pad1): track 18.8 -> 0.00 mm
- net Net-(C12-Pad2): track 16.6 -> 0.00 mm
- net /MOSI: track 15.5 -> 0.00 mm
- net Net-(D2-Pad2): track 14.2 -> 0.00 mm
- net Net-(C11-Pad2): track 13.8 -> 0.00 mm
- net Net-(J1-Pad2): track 12.6 -> 0.00 mm
- net Net-(J1-Pad1): track 10.8 -> 0.00 mm
- net Net-(J1-Pad3): track 9.12 -> 0.00 mm
- net Net-(R16-Pad2): track 8.77 -> 0.00 mm
- net /HV: track 9.72 -> 1.95 mm
- net Net-(C3-Pad2): track 0.00 -> 7.52 mm
- net /SCK: track 6.95 -> 0.00 mm
- net VCC: track 14.3 -> 7.93 mm
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Other:
- board size 67 x 21 mm -> 67 x 25 mm

Commit message: Recovery pdb start
Parts:
- added SW1: Test, Button_Switch_SMD:Panasonic_EVQPUJ_EVQPUA, F.Cu at (152.8, 103.2)
- BT1: footprint tester:batt -> Connector_PinHeader_2.54mm:PinHeader_1x02_P2.54mm_Vertical; moved to F.Cu
- C1, C10, C11, C13, C14, C15, C7: footprint Capacitors_SMD:C_0603 -> Resistor_SMD:R_0603_1608Metric
- C12, C8: footprint Capacitors_SMD:C_0603 -> Capacitor_SMD:C_0603_1608Metric
- C16, C3, C4, C5, C6: footprint Capacitors_SMD:C_0603 -> Resistor_SMD:R_0603_1608Metric; moved to F.Cu
- C9, U1, Y1: moved to F.Cu
- D2: footprint LEDs:LED_D3.0mm -> LED_THT:LED_D3.0mm; moved to F.Cu
- D3, Q1, Q3, Q4: footprint TO_SOT_Packages_SMD:SOT-23 -> Package_TO_SOT_SMD:SOT-23
- D4: footprint LEDs:LED_D3.0mm-3 -> LED_THT:LED_D3.0mm-3; moved to F.Cu
- D5, D7: footprint Diodes_SMD:D_MiniMELF_Standard -> Diode_SMD:D_MiniMELF
- D6: footprint Diodes_SMD:D_MiniMELF_Standard -> Diode_SMD:D_MiniMELF; moved to F.Cu
- J3: moved to B.Cu
- Q2, Q5, U7: footprint TO_SOT_Packages_SMD:SOT-23 -> Package_TO_SOT_SMD:SOT-23; moved to F.Cu
- R1, R2, R20, R23, R24, R27, R3, R4, R5, R6, R7: footprint Resistors_SMD:R_0603 -> Resistor_SMD:R_0603_1608Metric; moved to F.Cu
- R10, R11, R12, R13, R21, R22, R25, R26, R28, R29, R30, R8, R9: footprint Resistors_SMD:R_0603 -> Resistor_SMD:R_0603_1608Metric
- R14, R15, R16, R17, R18, R19: footprint Resistors_SMD:R_1206 -> Resistor_SMD:R_1206_3216Metric
- U2, U5: footprint TO_SOT_Packages_SMD:SOT-23-5 -> Package_TO_SOT_SMD:SOT-23-5
- U3: footprint Housings_QFP:TQFP-32_7x7mm_Pitch0.8mm -> Package_QFP:TQFP-32_7x7mm_P0.8mm
- U4: footprint TO_SOT_Packages_SMD:SOT-23-5 -> Package_TO_SOT_SMD:SOT-23-5; moved to F.Cu
- U6: footprint TO_SOT_Packages_SMD:SOT-23-6 -> Package_TO_SOT_SMD:SOT-23-6
- U8: footprint open-project:MICRO-B_USB -> Connector_USB:USB_Micro-B_Molex_47346-0001; moved to F.Cu
- moved C9 102.5 mm to (164.3, 69.4), turned to 0 degrees
- moved L1 100.4 mm to (168.5, 42.1), turned to 0 degrees
- moved D2 99.6 mm to (172.7, 61.7), turned to 0 degrees
- moved U5 93.4 mm to (166.2, 63.5), turned to 0 degrees
- moved D4 90.9 mm to (179.4, 32.9), turned to 0 degrees
- moved D1 88.0 mm to (182.0, 46.2)
- moved Q2 87.9 mm to (179.8, 53.8), turned to 0 degrees
- moved U4 82.2 mm to (180.6, 61.2), turned to 0 degrees
- moved BT1 81.1 mm to (192.1, 41.5), turned to 0 degrees
- moved U1 80.5 mm to (164.8, 34.9)
- moved D5 72.1 mm to (220.8, 32.0), turned to 0 degrees
- moved Q3 71.4 mm to (192.2, 56.4), turned to 0 degrees
- moved C7 71.1 mm to (160.5, 96.6), turned to 270 degrees
- moved L2 69.4 mm to (174.2, 42.4)
- moved Y1 69.3 mm to (176.5, 96.0)
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Routing:
- net GND: track 153.0 -> 22.3 mm, vias 1 -> 0
- net /SCK: track 0.00 -> 79.1 mm, vias 0 -> 1
- net /MOSI: track 0.00 -> 67.4 mm, vias 0 -> 1
- net /MISO: track 0.14 -> 66.0 mm, vias 0 -> 1
- net Net-(C7-Pad1): track 0.00 -> 56.8 mm, vias 0 -> 1
- net /RES: track 0.00 -> 52.9 mm, vias 0 -> 1
- net Net-(C15-Pad2): track 19.0 -> 0.00 mm
- net Net-(R14-Pad2): track 0.00 -> 14.2 mm
- net Net-(D1-Pad2): track 14.1 -> 0.00 mm
- net Net-(D4-Pad3): track 13.9 -> 0.00 mm
- net Net-(D6-Pad2): track 13.5 -> 0.00 mm
- net Net-(C14-Pad1): track 12.9 -> 0.00 mm
- net Net-(R16-Pad2): track 0.00 -> 12.9 mm
- net Net-(Q2-Pad1): track 12.6 -> 0.00 mm
- net Net-(R15-Pad2): track 0.00 -> 12.3 mm
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Other:
- board size 67 x 25 mm -> 73 x 20 mm

Commit message: Continue work with pcb
Parts:
- C1, C10, C13, C14, C15, C16, C3, C4, C5, C6, C7: footprint Resistor_SMD:R_0603_1608Metric -> Capacitor_SMD:C_0603_1608Metric
- U1: moved to B.Cu
- moved D4 71.6 mm to (205.2, 99.7), turned to 90 degrees
- moved R7 69.1 mm to (187.2, 98.4)
- moved R11 65.3 mm to (183.5, 102.4), turned to 180 degrees
- moved R13 63.3 mm to (187.2, 96.5)
- moved D6 59.1 mm to (202.3, 97.9), turned to 90 degrees
- moved R1 58.7 mm to (172.7, 88.8), turned to 90 degrees
- moved U1 56.9 mm to (173.2, 91.2)
- moved R6 56.8 mm to (187.2, 100.3), turned to 180 degrees
- moved C4 54.9 mm to (166.6, 86.2)
- moved R23 52.8 mm to (196.3, 101.1), turned to 90 degrees
- moved Q4 52.1 mm to (183.6, 99.6), turned to 90 degrees
- moved R24 51.9 mm to (194.1, 101.1), turned to 270 degrees
- moved C5 48.7 mm to (183.4, 87.0), turned to 90 degrees
- moved R2 48.6 mm to (174.5, 88.8), turned to 90 degrees
- moved Q2 46.9 mm to (190.9, 99.4), turned to 180 degrees
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Routing:
- net GND: track 22.3 -> 95.9 mm
- net Net-(D2-Pad2): track 5.25 -> 39.0 mm
- net Net-(Q4-Pad1): track 5.25 -> 35.6 mm
- net /D1: track 0.00 -> 29.4 mm
- net /D0: track 0.00 -> 29.1 mm
- net /D/C: track 0.00 -> 27.2 mm
- net /RS: track 0.00 -> 25.7 mm
- net Net-(C14-Pad1): track 0.00 -> 25.0 mm
- net Net-(Q5-Pad1): track 0.00 -> 10.0 mm
- net /+BATT: track 0.00 -> 9.46 mm
- net Net-(D6-Pad2): track 0.00 -> 9.16 mm
- net Net-(C6-Pad1): track 0.00 -> 8.20 mm, vias 0 -> 1
- net Net-(D4-Pad3): track 0.00 -> 7.68 mm
- net Net-(R4-Pad2): track 0.00 -> 7.37 mm, vias 0 -> 1
- net Net-(R2-Pad2): track 0.00 -> 7.05 mm, vias 0 -> 1
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
Commit message: Prefinal PCB
Parts:
- added J1: CONN_01X03_FEMALE, Connector_PinHeader_2.54mm:PinHeader_1x03_P2.54mm_Vertical, F.Cu at (135.4, 91.3)
- C11: footprint Resistor_SMD:R_0603_1608Metric -> Capacitor_SMD:C_0603_1608Metric
- C2, D1, L1, Q1, R10, U2: moved to B.Cu
- D4: value LED_Dual_ACAC -> LED_Dual_ACA
- L2: footprint w_smd_inductors:inductor_smd_4.8x2.8mm -> Inductor_SMD:L_0805_2012Metric
- moved C12 73.1 mm to (176.0, 98.3)
- moved D3 72.0 mm to (160.9, 102.3), turned to 90 degrees
- moved R12 67.8 mm to (147.2, 93.6), turned to 270 degrees
- moved R22 66.1 mm to (198.2, 101.6), turned to 180 degrees
- moved C13 65.7 mm to (164.2, 101.7)
- moved R25 65.4 mm to (198.2, 91.1), turned to 90 degrees
- moved C11 64.7 mm to (179.0, 98.3), turned to 180 degrees
- moved R9 63.7 mm to (188.0, 87.0), turned to 270 degrees
- moved D5 63.2 mm to (195.3, 89.8), turned to 90 degrees
- moved L1 61.0 mm to (200.9, 93.7), turned to 90 degrees
- moved C10 60.0 mm to (189.6, 87.0), turned to 90 degrees
- moved Q1 58.8 mm to (209.7, 90.9), turned to 270 degrees
- moved BT1 58.1 mm to (194.3, 99.6), turned to 180 degrees
- moved D1 49.2 mm to (205.7, 89.2), turned to 270 degrees
- moved L2 47.3 mm to (159.3, 87.3), turned to 270 degrees
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Connections:
- net Net-(J1-Pad1) renamed /IN_1
- net Net-(J1-Pad2) renamed /IN_2
- net Net-(J1-Pad3) renamed /IN_3
Routing:
- net GND: track 95.9 -> 268.3 mm, vias 0 -> 1
- net VCC: track 0.00 -> 124.3 mm, vias 0 -> 2
- net /HV: track 5.36 -> 93.4 mm, vias 0 -> 2
- net Net-(U3-Pad2): track 0.00 -> 77.8 mm
- net /BATT_TEST: track 0.00 -> 56.1 mm, vias 0 -> 1
- net Net-(C7-Pad1): track 59.3 -> 108.7 mm, vias 1 -> 2
- net Net-(R21-Pad2): track 0.00 -> 39.0 mm
- net Net-(Q4-Pad1): track 35.6 -> 6.77 mm
- net Net-(C13-Pad2): track 0.00 -> 26.9 mm
- net Net-(R8-Pad2): track 0.00 -> 26.2 mm, vias 0 -> 2
- net Net-(Q4-Pad3): track 4.06 -> 27.4 mm, vias 0 -> 2
- net /IN_1: track 7.50 -> 29.7 mm
- net /IN_2: track 8.48 -> 25.6 mm
- net Net-(C16-Pad1): track 0.00 -> 16.6 mm, vias 0 -> 1
- net /IN_3: track 8.49 -> 23.1 mm
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Other:
- net class Default: clearance 0.2 -> 0.1
- rule trace_clearance: 0.2 -> 0.1

Commit message: Final PCB
Parts:
- added J2: Probe1, tester:conn_tester, B.Cu at (141.3, 88.6)
- added J4: Probe2, tester:conn_tester, F.Cu at (141.3, 101.3)
- added J5: PAD, tester:conn_threepoint, F.Cu at (148.6, 89.2)
- C16: moved to B.Cu
- J1: value CONN_01X03_FEMALE -> FEMALE; footprint Connector_PinHeader_2.54mm:PinHeader_1x03_P2.54mm_Vertical -> Connector_PinSocket_2.54mm:PinSocket_1x03_P2.54mm_Vertical
- L1: footprint w_smd_inductors:inductor_smd_4.8x2.8mm -> Inductor_SMD:L_Coilcraft_XAL5030
- SW1: footprint Button_Switch_SMD:Panasonic_EVQPUJ_EVQPUA -> tester:BUT6120
- moved C16 14.6 mm to (186.8, 100.3)
- moved R10 10.7 mm to (154.7, 99.8), turned to 270 degrees
- moved SW1 8.95 mm to (148.9, 103.0), turned to 0 degrees
- moved J1 5.68 mm to (139.7, 95.0), turned to 90 degrees
- moved R12 3.86 mm to (150.0, 90.9), turned to 180 degrees
- moved R6 3.59 mm to (190.6, 102.2)
- moved R7 3.15 mm to (188.3, 101.5), turned to 270 degrees
- moved R13 2.87 mm to (186.9, 92.5), turned to 0 degrees
- moved R11 2.33 mm to (185.8, 102.9)
- moved Q4 2.18 mm to (185.7, 100.3)
- moved C12 1.59 mm to (174.6, 99.1)
- moved C11 1.51 mm to (177.7, 99.1)
- moved U6 1.18 mm to (150.6, 94.8)
- moved L1 0.09 mm to (201.0, 93.7), turned to 180 degrees
Connections:
- SW1 pad 1: Net-(D2-Pad2) -> Net-(Q4-Pad1)
- SW1 pad 2: Net-(Q4-Pad1) -> Net-(D2-Pad2)
Routing:
- net GND: track 268.3 -> 351.8 mm
- net Net-(D2-Pad2): track 30.0 -> 80.7 mm
- net Net-(Q4-Pad1): track 6.77 -> 43.5 mm
- net /IN_3: track 23.1 -> 48.4 mm
- net /IN_1: track 29.7 -> 52.7 mm
- net /IN_2: track 25.6 -> 44.7 mm
- net Net-(C16-Pad1): track 16.6 -> 33.6 mm
- net /RES: track 53.3 -> 65.6 mm
- net (no net): track 0.00 -> 10.8 mm
- net Net-(C7-Pad1): track 108.7 -> 104.7 mm
- net Net-(Q4-Pad3): track 27.4 -> 30.5 mm
- net VCC: track 124.3 -> 121.3 mm
- net /D1: track 31.5 -> 34.5 mm
- net /D0: track 30.4 -> 33.1 mm
- net /RS: track 29.4 -> 31.9 mm
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Other:
- board size 73 x 20 mm -> 75.1 x 20.1 mm
- board text added: "TESTER"

Commit message: Final correct and output
Parts:
- moved R4 5.08 mm to (173.0, 88.8)
- moved R1 4.57 mm to (177.0, 87.1), turned to 180 degrees
- moved R2 2.46 mm to (177.0, 88.8), turned to 180 degrees
- moved R3 1.89 mm to (177.0, 90.6), turned to 180 degrees
- moved R13 0.29 mm to (186.8, 92.2)
Connections:
- U3 pad 1: /RS -> /D1
- U3 pad 30: /D1 -> /RS
- U3 pad 31: /D0 -> /D/C
- U3 pad 32: /D/C -> /D0
Routing:
- net Net-(U3-Pad2): track 80.1 -> 85.8 mm
- net /RS: track 31.9 -> 37.2 mm
- net /D0: track 33.1 -> 28.6 mm
- net Net-(Q4-Pad1): track 43.5 -> 46.1 mm
- net /D1: track 34.5 -> 31.9 mm
- net Net-(R4-Pad2): track 7.37 -> 9.85 mm
- net /RES: track 65.6 -> 67.9 mm
- net Net-(R3-Pad2): track 6.92 -> 5.42 mm
- net GND: track 351.8 -> 353.0 mm
- net /D/C: track 32.2 -> 33.2 mm
- net Net-(R1-Pad2): track 6.58 -> 7.46 mm
Other:
- net class Default: via_dia 0.8 -> 1.2; via_drill 0.4 -> 0.2
