File: kicad/tester.sch (KiCad schematic (older format))
At the start: 73 parts, among them J1 CONN_01X03_FEMALE, J3 CONN_01X06, Q1 IRLML2402, Q2 IRLML6402, Q3 BC847, Q4 BC847, Q5 BC847, SW1 Test, U1 OLED_128x64, U2 NCP1450A, U3 ATMEGA328-AU, U4 LTC4054, U5 74LVC1G17, U6 SRV05, U7 XC6206P332, U8 MICRO-B_USB, Y1 16MHz

Commit message: Change package some resistors
Parts:
- R14, R15, R16, R17, R18, R19: footprint Resistors_SMD:R_0603 -> Resistors_SMD:R_1206
- U4: footprint TO_SOT_Packages_SMD:TSOT-23-5 -> TO_SOT_Packages_SMD:SOT-23-5
Changed lines of the file:
@@
 LIBS:Power_Management
 LIBS:tester_m
-LIBS:open-project
 LIBS:w_connectors
 LIBS:tester-cache
@@
 F 0 "R15" V 7050 900 50  0000 C CNN
 F 1 "470k" V 7050 1250 50  0000 C CNN
-F 2 "Resistors_SMD:R_0603" H 7100 1050 50  0001 C CNN
+F 2 "Resistors_SMD:R_1206" H 7100 1050 50  0001 C CNN
 F 3 "" H 7100 1050 50  0001 C CNN
 	1    7100 1050
@@
 F 0 "R17" V 7050 1100 50  0000 C CNN
 F 1 "470k" V 7050 1450 50  0000 C CNN
-F 2 "Resistors_SMD:R_0603" H 7100 1250 50  0001 C CNN
+F 2 "Resistors_SMD:R_1206" H 7100 1250 50  0001 C CNN
 F 3 "" H 7100 1250 50  0001 C CNN
 	1    7100 1250
@@
 F 0 "R19" V 7050 1300 50  0000 C CNN
 F 1 "470k" V 7050 1650 50  0000 C CNN
-F 2 "Resistors_SMD:R_0603" H 7100 1450 50  0001 C CNN
+F 2 "Resistors_SMD:R_1206" H 7100 1450 50  0001 C CNN
 F 3 "" H 7100 1450 50  0001 C CNN
 	1    7100 1450
@@
 F 0 "R14" V 7050 800 50  0000 C CNN
 F 1 "680" V 7050 1150 50  0000 C CNN
-F 2 "Resistors_SMD:R_0603" H 7100 950 50  0001 C CNN
+F 2 "Resistors_SMD:R_1206" H 7100 950 50  0001 C CNN
 F 3 "" H 7100 950 50  0001 C CNN
 	1    7100 950
@@
 F 0 "R16" V 7050 1000 50  0000 C CNN
 F 1 "680" V 7050 1350 50  0000 C CNN
-F 2 "Resistors_SMD:R_0603" H 7100 1150 50  0001 C CNN
+F 2 "Resistors_SMD:R_1206" H 7100 1150 50  0001 C CNN
 F 3 "" H 7100 1150 50  0001 C CNN
 	1    7100 1150
@@
 F 0 "R18" V 7050 1200 50  0000 C CNN
 F 1 "680" V 7050 1550 50  0000 C CNN
-F 2 "Resistors_SMD:R_0603" H 7100 1350 50  0001 C CNN
+F 2 "Resistors_SMD:R_1206" H 7100 1350 50  0001 C CNN
 F 3 "" H 7100 1350 50  0001 C CNN
 	1    7100 1350
@@
 F 0 "U4" H 6650 4613 60  0000 C CNN
 F 1 "LTC4054" H 6650 4719 60  0000 C CNN
-F 2 "TO_SOT_Packages_SMD:TSOT-23-5" H 6350 5250 60  0001 C CNN
+F 2 "TO_SOT_Packages_SMD:SOT-23-5" H 6350 5250 60  0001 C CNN
 F 3 "" H 6650 5000 60  0001 C CNN
 	1    6650 5000

Commit message: Add footprint oled
Parts:
- U1: footprint (none) -> tester:oled
Changed lines of the file:
@@
 LIBS:Power_Management
 LIBS:tester_m
+LIBS:open-project
 LIBS:w_connectors
 LIBS:tester-cache
@@
 F 0 "U1" H 1456 4187 60  0000 C CNN
 F 1 "OLED_128x64" H 1456 4081 60  0000 C CNN
-F 2 "" H 1350 1750 60  0001 C CNN
+F 2 "tester:oled" H 1350 1750 60  0001 C CNN
 F 3 "" H 1350 1750 60  0001 C CNN
 	1    1350 2450

Commit message: Update pcb
Parts:
- C5, C6: footprint (none) -> Capacitors_SMD:C_0603
- J3: footprint w_conn_jst-ph:s6b-ph-kl -> tester:avr_spi
Changed lines of the file:
@@
 F 0 "C5" V 2300 3700 50  0000 C CNN
 F 1 "2u2" V 2300 3500 50  0000 C CNN
-F 2 "" H 2250 3600 50  0001 C CNN
+F 2 "Capacitors_SMD:C_0603" H 2250 3600 50  0001 C CNN
 F 3 "" H 2250 3600 50  0001 C CNN
 	1    2250 3600
@@
 F 0 "C6" V 2350 3800 50  0000 C CNN
 F 1 "2u2" V 2350 3600 50  0000 C CNN
-F 2 "" H 2400 3700 50  0001 C CNN
+F 2 "Capacitors_SMD:C_0603" H 2400 3700 50  0001 C CNN
 F 3 "" H 2400 3700 50  0001 C CNN
 	1    2400 3700
@@
 F 0 "J3" H 10428 2991 50  0000 L CNN
 F 1 "CONN_01X06" H 10428 2900 50  0000 L CNN
-F 2 "w_conn_jst-ph:s6b-ph-kl" H 10350 2950 50  0001 C CNN
+F 2 "tester:avr_spi" H 10350 2950 50  0001 C CNN
 F 3 "" H 10350 2950 50  0001 C CNN
 	1    10350 2950

Commit message: Start pcb routing
Parts:
- BT1: footprint (none) -> tester:batt
- D4: footprint tester:led-dual-32x27 -> LEDs:LED_D3.0mm-3
- D5, D7: footprint (none) -> Diodes_SMD:D_MiniMELF_Standard
Connections:
- net labels added: +BATT
Changed lines of the file:
@@
 F 0 "BT1" H 4868 5246 50  0000 L CNN
 F 1 "Battery_Cell" H 4868 5155 50  0000 L CNN
-F 2 "" V 4750 5210 50  0001 C CNN
+F 2 "tester:batt" V 4750 5210 50  0001 C CNN
 F 3 "" V 4750 5210 50  0001 C CNN
 	1    4750 5150
@@
 F 0 "D5" V 8254 3029 50  0000 L CNN
 F 1 "5V1" V 8345 3029 50  0000 L CNN
-F 2 "" H 8300 2950 50  0001 C CNN
+F 2 "Diodes_SMD:D_MiniMELF_Standard" H 8300 2950 50  0001 C CNN
 F 3 "" H 8300 2950 50  0001 C CNN
 	1    8300 2950
@@
 F 0 "D7" H 9250 3884 50  0000 C CNN
 F 1 "5V1" H 9250 3975 50  0000 C CNN
-F 2 "" H 9250 4100 50  0001 C CNN
+F 2 "Diodes_SMD:D_MiniMELF_Standard" H 9250 4100 50  0001 C CNN
 F 3 "" H 9250 4100 50  0001 C CNN
 	1    9250 4100
@@
 F 0 "D4" H 7700 6283 50  0000 C CNN
 F 1 "LED_Dual_ACAC" H 7700 6374 50  0000 C CNN
-F 2 "tester:led-dual-32x27" H 7730 5950 50  0001 C CNN
+F 2 "LEDs:LED_D3.0mm-3" H 7730 5950 50  0001 C CNN
 F 3 "" H 7730 5950 50  0001 C CNN
 	1    7700 5950
@@
 Wire Wire Line
 	8750 6050 8000 6050
+Text Label 4850 4900 0    60   ~ 0
++BATT
 $EndSCHEMATC

Commit message: Continue work with pcb
Parts:
- D2: footprint (none) -> LEDs:LED_D3.0mm
Changed lines of the file:
@@
 LIBS:elec-unifil
 LIBS:gennum
-LIBS:graphic
 LIBS:hc11
 LIBS:intersil
@@
 LIBS:leds
 LIBS:LEM
-LIBS:logo
 LIBS:maxim
 LIBS:mechanical
@@
 F 0 "D2" H 5100 4050 50  0000 C CNN
 F 1 "LED_ALT" H 5000 4200 50  0000 C CNN
-F 2 "" H 4900 4100 50  0001 C CNN
+F 2 "LEDs:LED_D3.0mm" H 4900 4100 50  0001 C CNN
 F 3 "" H 4900 4100 50  0001 C CNN
 	1    4900 4100

Commit message: update pcb
Connections:
- wire segments 229 -> 231
Changed lines of the file:
@@
 L VCC #PWR038
 U 1 1 58E7E09A
-P 9750 900
-F 0 "#PWR038" H 9750 750 50  0001 C CNN
-F 1 "VCC" H 9700 1050 50  0000 L CNN
-F 2 "" H 9750 900 50  0001 C CNN
-F 3 "" H 9750 900 50  0001 C CNN
-	1    9750 900
+P 9800 900
+F 0 "#PWR038" H 9800 750 50  0001 C CNN
+F 1 "VCC" H 9750 1050 50  0000 L CNN
+F 2 "" H 9800 900 50  0001 C CNN
+F 3 "" H 9800 900 50  0001 C CNN
+	1    9800 900
 	1    0    0    -1
 $EndComp
@@
 	1    0    0    -1
 $EndComp
-$Comp
-L VCC #PWR045
-U 1 1 58EA6E48
-P 9800 2550
-F 0 "#PWR045" H 9800 2400 50  0001 C CNN
-F 1 "VCC" H 9800 2700 50  0000 L CNN
-F 2 "" H 9800 2550 50  0001 C CNN
-F 3 "" H 9800 2550 50  0001 C CNN
-	1    9800 2550
-	1    0    0    -1
-$EndComp
 Text Label 9900 3000 0    60   ~ 0
 MOSI
@@
 	10150 2900 9900 2900
 Wire Wire Line
-	9800 2800 9800 2550
-Wire Wire Line
-	10150 2800 9800 2800
+	9600 600  9600 2800
+Wire Wire Line
+	9600 2800 10150 2800
 Wire Wire Line
 	10150 2700 9900 2700
@@
 	10150 1000 10150 900
 Wire Wire Line
-	9750 1000 10150 1000
-Wire Wire Line
-	9750 900  9750 1000
+	9800 1000 10150 1000
+Wire Wire Line
+	9800 900  9800 1000
 Wire Wire Line
 	10650 1050 10650 900
@@
 Text Label 4850 4900 0    60   ~ 0
 +BATT
+Wire Wire Line
+	9600 600  3500 600
+Wire Wire Line
+	3500 600  3500 950
+Connection ~ 3500 950
 $EndSCHEMATC

Commit message: Working with pcb
Connections:
- wire segments 231 -> 298

Commit message: Recovery pdb start
Parts:
- BT1: footprint tester:batt -> Connector_PinHeader_2.54mm:PinHeader_1x02_P2.54mm_Vertical; symbol Battery_Cell -> tester-rescue:Battery_Cell
- C1, C10, C11, C13, C14, C15, C16, C3, C4, C5, C6, C7: footprint Capacitors_SMD:C_0603 -> Resistor_SMD:R_0603_1608Metric; symbol C_Small -> tester-rescue:C_Small
- C12, C8: footprint Capacitors_SMD:C_0603 -> Capacitor_SMD:C_0603_1608Metric; symbol C_Small -> tester-rescue:C_Small
- C2, C9: symbol CP_Small -> tester-rescue:CP_Small
- D1: symbol SM5819 -> tester_m:SM5819
- D2: footprint LEDs:LED_D3.0mm -> LED_THT:LED_D3.0mm; symbol LED_ALT -> tester-rescue:LED_ALT
- D3: footprint TO_SOT_Packages_SMD:SOT-23 -> Package_TO_SOT_SMD:SOT-23; symbol TL431DBZ -> tester-rescue:TL431DBZ
- D4: footprint LEDs:LED_D3.0mm-3 -> LED_THT:LED_D3.0mm-3; symbol LED_Dual_ACAC -> tester-rescue:LED_Dual_ACAC
- D5, D7: footprint Diodes_SMD:D_MiniMELF_Standard -> Diode_SMD:D_MiniMELF; symbol D_Zener -> tester-rescue:D_Zener
- D6: footprint Diodes_SMD:D_MiniMELF_Standard -> Diode_SMD:D_MiniMELF; symbol LL4148 -> tester-rescue:LL4148
- J1: symbol CONN_01X03_FEMALE -> tester-rescue:CONN_01X03_FEMALE
- J3: symbol CONN_01X06 -> tester-rescue:CONN_01X06
- L1: symbol L_Core_Iron -> tester-rescue:L_Core_Iron
- L2: symbol L -> tester-rescue:L
- Q1: footprint TO_SOT_Packages_SMD:SOT-23 -> Package_TO_SOT_SMD:SOT-23; symbol IRLML2402 -> tester_m:IRLML2402
- Q2: footprint TO_SOT_Packages_SMD:SOT-23 -> Package_TO_SOT_SMD:SOT-23; symbol IRLML6402 -> tester_m:IRLML6402
- Q3, Q4, Q5: footprint TO_SOT_Packages_SMD:SOT-23 -> Package_TO_SOT_SMD:SOT-23; symbol BC847 -> tester-rescue:BC847
- R1, R10, R11, R12, R13, R2, R20, R21, R22, R23, R24, R25, R26, R27, R28, R29, R3, R30, R4, R5, R6, R7, R8, R9: footprint Resistors_SMD:R_0603 -> Resistor_SMD:R_0603_1608Metric; symbol R_Small -> tester-rescue:R_Small
- R14, R15, R16, R17, R18, R19: footprint Resistors_SMD:R_1206 -> Resistor_SMD:R_1206_3216Metric; symbol R_Small -> tester-rescue:R_Small
- SW1: footprint (none) -> Button_Switch_SMD:Panasonic_EVQPUJ_EVQPUA; symbol SW_Push -> tester-rescue:SW_Push
- U1: symbol OLED_128x64 -> tester_m:OLED_128x64
- U2: footprint TO_SOT_Packages_SMD:SOT-23-5 -> Package_TO_SOT_SMD:SOT-23-5; symbol NCP1450A -> tester_m:NCP1450A
- U3: footprint Housings_QFP:TQFP-32_7x7mm_Pitch0.8mm -> Package_QFP:TQFP-32_7x7mm_P0.8mm; symbol ATMEGA328-AU -> tester-rescue:ATMEGA328-AU
- U4: footprint TO_SOT_Packages_SMD:SOT-23-5 -> Package_TO_SOT_SMD:SOT-23-5; symbol LTC4054 -> tester_m:LTC4054
- U5: footprint TO_SOT_Packages_SMD:SOT-23-5 -> Package_TO_SOT_SMD:SOT-23-5; symbol 74LVC1G17 -> tester-rescue:74LVC1G17
- U6: footprint TO_SOT_Packages_SMD:SOT-23-6 -> Package_TO_SOT_SMD:SOT-23-6; symbol SRV05 -> tester-rescue:SRV05
- U7: footprint TO_SOT_Packages_SMD:SOT-23 -> Package_TO_SOT_SMD:SOT-23; symbol XC6206P332 -> tester_m:XC6206P332
- U8: footprint open-project:MICRO-B_USB -> Connector_USB:USB_Micro-B_Molex_47346-0001; symbol MICRO-B_USB -> tester-rescue:MICRO-B_USB
- Y1: symbol Crystal_Small -> tester-rescue:Crystal_Small
