File: kicad/tester.sch (KiCad schematic (older format))
At the start: 73 parts, among them J1 CONN_01X03_FEMALE, J3 CONN_01X06, Q1 IRLML2402, Q2 IRLML6402, Q3 BC847, Q4 BC847, Q5 BC847, SW1 Test, U1 OLED_128x64, U2 NCP1450A, U3 ATMEGA328-AU, U4 LTC4054, U5 74LVC1G17, U6 SRV05, U7 XC6206P332, U8 MICRO-B_USB, Y1 16MHz

Commit message: Continue work with pcb
Parts:
- C1, C10, C13, C14, C15, C16, C3, C4, C5, C6, C7: footprint Resistor_SMD:R_0603_1608Metric -> Capacitor_SMD:C_0603_1608Metric
Changed lines of the file:
@@
 F 0 "C7" V 3100 1150 50  0000 C CNN
 F 1 "0.1u" V 3100 1400 50  0000 C CNN
-F 2 "Resistor_SMD:R_0603_1608Metric" H 3150 1250 50  0001 C CNN
+F 2 "Capacitor_SMD:C_0603_1608Metric" H 3150 1250 50  0001 C CNN
 F 3 "" H 3150 1250 50  0001 C CNN
 	1    3150 1250
@@
 F 0 "C13" V 6600 2250 50  0000 C CNN
 F 1 "0.1u" V 6600 2500 50  0000 C CNN
-F 2 "Resistor_SMD:R_0603_1608Metric" H 6650 2350 50  0001 C CNN
+F 2 "Capacitor_SMD:C_0603_1608Metric" H 6650 2350 50  0001 C CNN
 F 3 "" H 6650 2350 50  0001 C CNN
 	1    6650 2350
@@
 F 0 "C3" V 2100 1200 50  0000 C CNN
 F 1 "1u" V 2100 1000 50  0000 C CNN
-F 2 "Resistor_SMD:R_0603_1608Metric" H 2050 1100 50  0001 C CNN
+F 2 "Capacitor_SMD:C_0603_1608Metric" H 2050 1100 50  0001 C CNN
 F 3 "" H 2050 1100 50  0001 C CNN
 	1    2050 1100
@@
 F 0 "C4" V 2100 1400 50  0000 C CNN
 F 1 "1u" V 2100 1200 50  0000 C CNN
-F 2 "Resistor_SMD:R_0603_1608Metric" H 2050 1300 50  0001 C CNN
+F 2 "Capacitor_SMD:C_0603_1608Metric" H 2050 1300 50  0001 C CNN
 F 3 "" H 2050 1300 50  0001 C CNN
 	1    2050 1300
@@
 F 0 "C5" V 2300 3700 50  0000 C CNN
 F 1 "2u2" V 2300 3500 50  0000 C CNN
-F 2 "Resistor_SMD:R_0603_1608Metric" H 2250 3600 50  0001 C CNN
+F 2 "Capacitor_SMD:C_0603_1608Metric" H 2250 3600 50  0001 C CNN
 F 3 "" H 2250 3600 50  0001 C CNN
 	1    2250 3600
@@
 F 0 "C6" V 2350 3800 50  0000 C CNN
 F 1 "2u2" V 2350 3600 50  0000 C CNN
-F 2 "Resistor_SMD:R_0603_1608Metric" H 2400 3700 50  0001 C CNN
+F 2 "Capacitor_SMD:C_0603_1608Metric" H 2400 3700 50  0001 C CNN
 F 3 "" H 2400 3700 50  0001 C CNN
 	1    2400 3700
@@
 F 0 "C1" H 1300 5050 50  0000 C CNN
 F 1 "0.1u" H 1250 4850 50  0000 C CNN
-F 2 "Resistor_SMD:R_0603_1608Metric" H 1350 4950 50  0001 C CNN
+F 2 "Capacitor_SMD:C_0603_1608Metric" H 1350 4950 50  0001 C CNN
 F 3 "" H 1350 4950 50  0001 C CNN
 	1    1350 4950
@@
 F 0 "C10" H 5750 4600 50  0000 C CNN
 F 1 "0.01" H 5750 4400 50  0000 C CNN
-F 2 "Resistor_SMD:R_0603_1608Metric" H 5850 4500 50  0001 C CNN
+F 2 "Capacitor_SMD:C_0603_1608Metric" H 5850 4500 50  0001 C CNN
 F 3 "" H 5850 4500 50  0001 C CNN
 	1    5850 4500
@@
 F 0 "C14" H 7458 5296 50  0000 R CNN
 F 1 "0.1u" H 7458 5205 50  0000 R CNN
-F 2 "Resistor_SMD:R_0603_1608Metric" H 7550 5250 50  0001 C CNN
+F 2 "Capacitor_SMD:C_0603_1608Metric" H 7550 5250 50  0001 C CNN
 F 3 "" H 7550 5250 50  0001 C CNN
 	1    7550 5250
@@
 F 0 "C15" V 8150 4300 50  0000 C CNN
 F 1 "0.1" V 8150 4550 50  0000 C CNN
-F 2 "Resistor_SMD:R_0603_1608Metric" H 8200 4400 50  0001 C CNN
+F 2 "Capacitor_SMD:C_0603_1608Metric" H 8200 4400 50  0001 C CNN
 F 3 "" H 8200 4400 50  0001 C CNN
 	1    8200 4400
@@
 F 0 "C16" H 2959 4146 50  0000 R CNN
 F 1 "1u" H 2959 4055 50  0000 R CNN
-F 2 "Resistor_SMD:R_0603_1608Metric" H 3050 4100 50  0001 C CNN
+F 2 "Capacitor_SMD:C_0603_1608Metric" H 3050 4100 50  0001 C CNN
 F 3 "" H 3050 4100 50  0001 C CNN
 	1    3050 4100

Commit message: Prefinal PCB
Parts:
- removed D4: LED_Dual_ACAC, LED_THT:LED_D3.0mm-3, symbol tester-rescue:LED_Dual_ACAC
- added D4: LED_Dual_ACA, LED_THT:LED_D3.0mm-3, symbol Device:LED_Dual_ACA
- C11: footprint Resistor_SMD:R_0603_1608Metric -> Capacitor_SMD:C_0603_1608Metric
- J1: footprint (none) -> Connector_PinHeader_2.54mm:PinHeader_1x03_P2.54mm_Vertical
- L2: footprint w_smd_inductors:inductor_smd_4.8x2.8mm -> Inductor_SMD:L_0805_2012Metric
Connections:
- net GND: now also D4.2 (K)
- net IN_1: now reaches J1.1, R14.1, R15.1, U3.23 ((PCINT8/ADC0)PC0), U6.4 (COM3)
- net IN_2: now reaches J1.2, R16.1, R17.1, U3.24 ((PCINT9/ADC1)PC1), U6.6 (COM4)
- net IN_3: now reaches J1.3, R18.1, R19.1, U3.25 ((PCINT10/ADC2)PC2), U6.1 (COM1)
- net at Q5.2 (E): now also D4.3 (A2)
- net at D6.1 (K): now also D4.1 (A1)
Changed lines of the file:
@@
 F 0 "L2" V 3340 1050 50  0000 C CNN
 F 1 "10uH" V 3249 1050 50  0000 C CNN
-F 2 "w_smd_inductors:inductor_smd_4.8x2.8mm" H 3150 1050 50  0001 C CNN
+F 2 "Inductor_SMD:L_0805_2012Metric" H 3150 1050 50  0001 C CNN
 F 3 "" H 3150 1050 50  0001 C CNN
 	1    3150 1050
@@
 F 0 "C11" V 6350 1450 50  0000 C CNN
 F 1 "22pF" V 6350 1700 50  0000 C CNN
-F 2 "Resistor_SMD:R_0603_1608Metric" H 6400 1550 50  0001 C CNN
+F 2 "Capacitor_SMD:C_0603_1608Metric" H 6400 1550 50  0001 C CNN
 F 3 "" H 6400 1550 50  0001 C CNN
 	1    6400 1550
@@
 F 0 "J1" H 9478 1841 50  0000 L CNN
 F 1 "CONN_01X03_FEMALE" H 9478 1750 50  0000 L CNN
-F 2 "" H 9300 2000 50  0001 C CNN
+F 2 "Connector_PinHeader_2.54mm:PinHeader_1x03_P2.54mm_Vertical" H 9300 2000 50  0001 C CNN
 F 3 "" H 9300 2000 50  0001 C CNN
 	1    9300 1800
@@
 Wire Wire Line
 	3400 3250 3400 3400
-$Comp
-L tester-rescue:LED_Dual_ACAC D4
-U 1 1 58EA8262
-P 7700 5950
-F 0 "D4" H 7700 6283 50  0000 C CNN
-F 1 "LED_Dual_ACAC" H 7700 6374 50  0000 C CNN
-F 2 "LED_THT:LED_D3.0mm-3" H 7730 5950 50  0001 C CNN
-F 3 "" H 7730 5950 50  0001 C CNN
-	1    7700 5950
-	-1   0    0    1
-$EndComp
-Wire Wire Line
-	7350 5850 7350 5950
-Wire Wire Line
-	7350 5950 7350 6050
-Connection ~ 7350 5950
-Wire Wire Line
-	7250 5950 7350 5950
-Wire Wire Line
-	7400 5850 7350 5850
-Wire Wire Line
-	7350 6050 7400 6050
-Wire Wire Line
-	8300 5850 8000 5850
-Wire Wire Line
-	8750 6050 8000 6050
 Text Label 4850 4900 0    60   ~ 0
 +BATT
@@
 	3500 600  3500 950
 Connection ~ 3500 950
+Text Label 8750 1600 0    50   ~ 0
+IN_1
+Text Label 8750 1800 0    50   ~ 0
+IN_2
+Text Label 8750 2000 0    50   ~ 0
+IN_3
+$Comp
+L Device:LED_Dual_ACA D4
+U 1 1 5ABA3E73
+P 7700 5950
+F 0 "D4" H 7450 6050 50  0000 C CNN
+F 1 "LED_Dual_ACA" H 7750 5700 50  0000 C CNN
+F 2 "LED_THT:LED_D3.0mm-3" H 7700 5950 50  0001 C CNN
+F 3 "~" H 7700 5950 50  0001 C CNN
+	1    7700 5950
+	1    0    0    1
+$EndComp
+Wire Wire Line
+	7400 5950 7250 5950
+Wire Wire Line
+	8000 5850 8300 5850
+Wire Wire Line
+	8750 6050 8000 6050
 $EndSCHEMATC

Commit message: Final PCB
Parts:
- removed SW1: Test, Button_Switch_SMD:Panasonic_EVQPUJ_EVQPUA, symbol tester-rescue:SW_Push
- added J2: Probe1, tester:conn_tester, symbol Connector_Generic:Conn_01x02
- added J4: Probe2, tester:conn_tester, symbol Connector_Generic:Conn_01x02
- added J5: PAD, tester:conn_threepoint, symbol Connector_Generic:Conn_01x03
- added SW1: Test, tester:BUT6120, symbol Switch:SW_Push_Dual
- J1: value CONN_01X03_FEMALE -> FEMALE; footprint Connector_PinHeader_2.54mm:PinHeader_1x03_P2.54mm_Vertical -> Connector_PinSocket_2.54mm:PinSocket_1x03_P2.54mm_Vertical
- L1: footprint w_smd_inductors:inductor_smd_4.8x2.8mm -> Inductor_SMD:L_Coilcraft_XAL5030
Connections:
- net GND: now also J2.2 (Pin_2), J4.2 (Pin_2), SW1.3
- net IN_1: now also J2.1 (Pin_1), J5.1 (Pin_1)
- net IN_2: now also J5.2 (Pin_2)
- net IN_3: now also J4.1 (Pin_1), J5.3 (Pin_3)
- net at D2.2 (A), R6.2: now also SW1.2
- net at Q4.1 (B), R11.2: now also SW1.1
- no-connect marks 8 -> 9
Changed lines of the file:
@@
 F 0 "L1" V 2825 4600 50  0000 C CNN
 F 1 "10uH" V 2734 4600 50  0000 C CNN
-F 2 "w_smd_inductors:inductor_smd_4.8x2.8mm" H 2600 4600 50  0001 C CNN
+F 2 "Inductor_SMD:L_Coilcraft_XAL5030" H 2600 4600 50  0001 C CNN
 F 3 "" H 2600 4600 50  0001 C CNN
 	1    2600 4600
@@
 $EndComp
 $Comp
-L tester-rescue:SW_Push SW1
-U 1 1 58E71041
-P 4950 3800
-F 0 "SW1" H 4650 3850 50  0000 C CNN
-F 1 "Test" H 5200 3850 50  0000 C CNN
-F 2 "Button_Switch_SMD:Panasonic_EVQPUJ_EVQPUA" H 4950 4000 50  0001 C CNN
-F 3 "" H 4950 4000 50  0001 C CNN
-	1    4950 3800
-	1    0    0    -1
-$EndComp
-$Comp
 L tester-rescue:Battery_Cell BT1
 U 1 1 58E71A72
@@
 P 9300 1800
 F 0 "J1" H 9478 1841 50  0000 L CNN
-F 1 "CONN_01X03_FEMALE" H 9478 1750 50  0000 L CNN
-F 2 "Connector_PinHeader_2.54mm:PinHeader_1x03_P2.54mm_Vertical" H 9300 2000 50  0001 C CNN
+F 1 "FEMALE" H 9650 1750 50  0000 L CNN
+F 2 "Connector_PinSocket_2.54mm:PinSocket_1x03_P2.54mm_Vertical" H 9300 2000 50  0001 C CNN
 F 3 "" H 9300 2000 50  0001 C CNN
 	1    9300 1800
@@
 F 3 "" H 8300 2950 50  0001 C CNN
 	1    8300 2950
-	0    1    1    0
+	0    -1   1    0
 $EndComp
 $Comp
@@
 	8400 1900 8400 1800
 Wire Wire Line
-	8400 1800 9200 1800
+	8400 1800 8600 1800
 Connection ~ 7600 1600
 Wire Wire Line
-	7600 1600 9200 1600
+	7600 1600 8700 1600
 Connection ~ 4750 4900
 Wire Wire Line
 	4750 5300 4750 5250
 Connection ~ 6350 3500
-Wire Wire Line
-	6100 3800 6100 3500
-Wire Wire Line
-	5150 3800 6100 3800
 Connection ~ 4450 4100
-Wire Wire Line
-	4750 3800 4450 3800
 Wire Wire Line
 	6700 2950 6700 3000
@@
 	5650 4350 5650 4400
 Wire Wire Line
-	4450 3800 4450 4100
-Wire Wire Line
 	4450 4100 4450 4300
 Wire Wire Line
@@
 	3150 1400 3150 3650
 Wire Wire Line
-	3150 3650 6000 3650
-Wire Wire Line
-	6000 3650 6000 2400
+	3150 3650 3900 3650
 Wire Wire Line
 	6000 2400 5950 2400
@@
 Connection ~ 4150 4600
 Wire Wire Line
-	8600 3950 4150 3950
-Wire Wire Line
-	8600 2100 8600 3950
-Wire Wire Line
-	7850 2100 8600 2100
+	8400 3950 4150 3950
+Wire Wire Line
+	8400 2100 8400 3950
+Wire Wire Line
+	7850 2100 8400 2100
 Wire Wire Line
 	2350 5100 2350 5300
@@
 	5450 2000 7400 2000
 Wire Wire Line
-	7400 2000 9200 2000
+	7400 2000 8500 2000
 Wire Wire Line
 	7400 1350 7400 1450
@@
 Wire Wire Line
 	8750 6050 8000 6050
+$Comp
+L Connector_Generic:Conn_01x02 J2
+U 1 1 5AC1877C
+P 9400 1250
+F 0 "J2" H 9480 1242 50  0000 L CNN
+F 1 "Probe1" H 9300 1050 50  0000 L CNN
+F 2 "tester:conn_tester" H 9400 1250 50  0001 C CNN
+F 3 "~" H 9400 1250 50  0001 C CNN
+	1    9400 1250
+	1    0    0    -1
+$EndComp
+$Comp
+L Connector_Generic:Conn_01x02 J4
+U 1 1 5AC189EA
+P 9300 2200
+F 0 "J4" H 9380 2192 50  0000 L CNN
+F 1 "Probe2" H 9300 1950 50  0000 L CNN
+F 2 "tester:conn_tester" H 9300 2200 50  0001 C CNN
+F 3 "~" H 9300 2200 50  0001 C CNN
+	1    9300 2200
+	1    0    0    -1
+$EndComp
+$Comp
+L tester-rescue:GND-RESCUE-tester #PWR0101
+U 1 1 5AC18B99
+P 9150 1400
+F 0 "#PWR0101" H 9150 1150 50  0001 C CNN
+F 1 "GND" H 9155 1227 50  0000 C CNN
+F 2 "" H 9150 1400 50  0001 C CNN
+F 3 "" H 9150 1400 50  0001 C CNN
+	1    9150 1400
+	1    0    0    -1
+$EndComp
+$Comp
+L tester-rescue:GND-RESCUE-tester #PWR0102
+U 1 1 5AC18C3A
+P 9050 2350
+F 0 "#PWR0102" H 9050 2100 50  0001 C CNN
+F 1 "GND" H 9055 2177 50  0000 C CNN
+F 2 "" H 9050 2350 50  0001 C CNN
+F 3 "" H 9050 2350 50  0001 C CNN
+	1    9050 2350
+	1    0    0    -1
+$EndComp
+Wire Wire Line
+	9050 2350 9050 2300
+Wire Wire Line
+	9050 2300 9100 2300
+Wire Wire Line
+	9150 1400 9150 1350
+Wire Wire Line
+	9150 1350 9200 1350
+Connection ~ 9050 1600
+Wire Wire Line
+	9050 1600 9200 1600
+Connection ~ 9050 2000
+Wire Wire Line
+	9050 2000 9200 2000
+$Comp
+L Connector_Generic:Conn_01x03 J5
+U 1 1 5AC28CE1
+P 8950 2750
+F 0 "J5" H 9030 2792 50  0000 L CNN
+F 1 "PAD" H 9030 2701 50  0000 L CNN
+F 2 "tester:conn_threepoint" H 8950 2750 50  0001 C CNN
+F 3 "~" H 8950 2750 50  0001 C CNN
+	1    8950 2750
+	1    0    0    -1
+$EndComp
+Wire Wire Line
+	8750 2650 8700 2650
+Wire Wire Line
+	8700 2650 8700 1600
+Connection ~ 8700 1600
+Wire Wire Line
+	8700 1600 9050 1600
+Wire Wire Line
+	8750 2750 8600 2750
+Wire Wire Line
+	8600 2750 8600 1800
+Connection ~ 8600 1800
+Wire Wire Line
+	8600 1800 9200 1800
+Wire Wire Line
+	8750 2850 8500 2850
+Wire Wire Line
+	8500 2850 8500 2000
+Connection ~ 8500 2000
+Wire Wire Line
+	8500 2000 9050 2000
+Wire Wire Line
+	9050 2200 9100 2200
+Wire Wire Line
+	9050 2000 9050 2200
+Wire Wire Line
+	9200 1250 9050 1250
+Wire Wire Line
+	9050 1250 9050 1600
+Wire Wire Line
+	3900 3650 3900 3450
+Wire Wire Line
+	3900 3450 6000 3450
+Wire Wire Line
+	6000 3450 6000 2400
+Wire Wire Line
+	4450 3600 4450 4100
+Wire Wire Line
+	4450 3600 4750 3600
+Wire Wire Line
+	5150 3600 6100 3600
+Wire Wire Line
+	6100 3600 6100 3500
+$Comp
+L Switch:SW_Push_Dual SW1
+U 1 1 5AE7EFF2
+P 4950 3600
+F 0 "SW1" H 4500 3650 50  0000 C CNN
+F 1 "Test" H 5250 3650 50  0000 C CNN
+F 2 "tester:BUT6120" H 4950 3800 50  0001 C CNN
+F 3 "" H 4950 3800 50  0001 C CNN
+	1    4950 3600
+	-1   0    0    -1
+$EndComp
+$Comp
+L tester-rescue:GND-RESCUE-tester #PWR?
+U 1 1 5B1BE9C1
+P 5250 3800
+F 0 "#PWR?" H 5250 3550 50  0001 C CNN
+F 1 "GND" H 5255 3627 50  0000 C CNN
+F 2 "" H 5250 3800 50  0001 C CNN
+F 3 "" H 5250 3800 50  0001 C CNN
+	1    5250 3800
+	0    -1   -1   0
+$EndComp
+Wire Wire Line
+	5150 3800 5250 3800
+NoConn ~ 4750 3800
 $EndSCHEMATC

Commit message: Final correct and output
Connections:
- net D/C: now also U3.31 ((PCINT17/TXD)PD1); no longer U3.32 ((PCINT18/INT0)PD2)
- net D0: now also U3.32 ((PCINT18/INT0)PD2); no longer U3.31 ((PCINT17/TXD)PD1)
- net D1: now also U3.1 ((PCINT19/OC2B/INT1)PD3); no longer U3.30 ((PCINT16/RXD)PD0)
- net RS: now also U3.30 ((PCINT16/RXD)PD0); no longer U3.1 ((PCINT19/OC2B/INT1)PD3)
Other:
- note added: "SCLK"
- note added: "SDIN"
Changed lines of the file:
@@
 Text Label 2800 2800 0    60   ~ 0
 D1
+Text Label 5700 2550 0    60   ~ 0
+RS
+Text Label 5700 2650 0    60   ~ 0
+D/C
+Text Label 5700 2750 0    60   ~ 0
+D0
 Text Label 5700 2850 0    60   ~ 0
-RS
-Text Label 5700 2750 0    60   ~ 0
-D/C
-Text Label 5700 2650 0    60   ~ 0
-D0
-Text Label 5700 2550 0    60   ~ 0
 D1
 $Comp
@@
 	5150 3800 5250 3800
 NoConn ~ 4750 3800
+Text Notes 2600 2700 0    50   ~ 0
+SCLK
+Text Notes 2600 2800 0    50   ~ 0
+SDIN
 $EndSCHEMATC
